File: eagle/iTrope/itrope-serial-v05.brd (EAGLE design)
At the start: 30.5 x 28.5 mm, 30 parts, among them IC1 78L05Z, J1 ITRIP-V1, U1 FT232RL-BASICSSOP, X1 22-23-2021, X10 87758-0216, X2 22-23-2021, X3 22-23-2021, X4 22-23-2021, X5 87758-0216, X6 22-23-2031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

Commit message: tweak eagle board and sundries
Parts:
- turned X1 to 90 degrees
- turned X2 to 90 degrees
Routing:
- net RXD: track 42.8 -> 40.0 mm
- net TXD: track 45.3 -> 47.0 mm
- net +3V3: track 50.6 -> 51.7 mm
